File: 0000.0108.kicad_sch (KiCad schematic)
At the start: 108 parts, among them J1 XA, J10 NC3FAAH, J11 XA, J13 XH, J2 XA, J3 XA, J4 XA, J5 XA, J6 TMT152xx, J7 RAC10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

Commit message: Updated missing or ambiguous component values. Added feed resistor bypass links.
Parts:
- added JP1, JP2: blob, Jumper:SolderJumper-2_P1.3mm_Open_RoundedPad1.0x1.5mm, symbol Jumper:SolderJumper_2_Open
- J1, J11, J2, J3, J4, J5: value XA -> B3B-XH-A
- J13: value XH -> B4B-XH-A
- J6: value TMT152xx -> TMT15215; now not fitted
- J7: value RAC10 -> RAC10-15DK/277
- J8: value JH -> B2P3 -VH
- L1, L2, L3, L4: value 10 -> 10.1210
- L7, L8: value 10 -> 10.4x4
- R14, R31: value 1K -> 3K3
- R26, R9: value 7K5 -> 5K6
Connections:
- net OUT1: now also JP1.1 (A)
- net OUT2: now also JP2.1 (A)
- net at J2.1 (Pin_1), R34.2: now also JP1.2 (B)
- net at J2.3 (Pin_3), R36.2: now also JP2.2 (B)
Other:
- moved on the sheet: C11, C12, C25, C26, C27, C28, C29, C30, C31, C32, F1, H1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

Commit message: Changed XLR input connectors from NC3FAH to NC3FAH2 as the latter is compatible with both. NC3FAH has the shield/screw contact connected to pin 1. NC3FAH2 has this as a separate fourth pin.
Parts:
- removed J10, J9: NC3FAAH, Connector_Audio:Jack_XLR_Neutrik_NC3FAAH_Horizontal, symbol Connector_Audio:NC3FAAH
- added J10, J9: NC3FAAH2, Connector_Audio:Jack_XLR_Neutrik_NC3FAAH2_Horizontal, symbol Connector_Audio:NC3FAAH2
- J6: footprint HR_Parts:PSU_TRACO_TMT152xx -> HR_parts:PSU_TRACO_TMT152xx
- J7: footprint HR_Parts:RECOM-RAC10 -> HR_parts:RECOM-RAC10
- L7, L8: footprint HR_Parts:INDUCTOR_SMD_4x4 -> HR_parts:INDUCTOR_SMD_4x4
Connections:
- net GND: now also J10.1, J10.G, J9.1, J9.G
- net at C19.1, J5.1 (Pin_1), R18.1: now also J10.2
- net at C20.1, J5.3 (Pin_3), R19.2: now also J10.3
- net at C6.1, J4.3 (Pin_3), R8.2: now also J9.3
- net at C5.1, J4.1 (Pin_1), R7.1: now also J9.2
